File: Circuits/Eagle/Input.brd (EAGLE design)
At the start: 42.8 x 80 mm, 7 parts

Commit message: KiCAD,EAGLEでのPCB設計を試行中。
Parts:
- removed C1: 0.22F, capacitor-wima:C2.5-3
Connections:
- removed net N$1: C1.2, G1.-, JP1.2, U$1.P$28
- new net N$10: JP1.2, U$1.P$28
- net N$3: no longer C1.1, G1.+
Changed lines of the file:
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@@
 </autorouter>
 <elements>
-<element name="C1" library="capacitor-wima" package="C2.5-3" value="0.22F" x="-16.51" y="52.07"/>
 <element name="G1" library="battery" package="CR2032H" value="CR2032H" x="-22.86" y="10.16"/>
 <element name="JP1" library="pinhead" package="1X02" value="CFG" x="-38.1" y="44.45"/>
@@
 </elements>
 <signals>
-<signal name="N$1">
-<contactref element="C1" pad="2"/>
-<contactref element="U$1" pad="P$28"/>
-<contactref element="G1" pad="-"/>
-<contactref element="JP1" pad="2"/>
-<wire x1="-20.32" y1="39.12" x2="-15.24" y2="52.07" width="0" layer="19" extent="1-1"/>
-<wire x1="-36.83" y1="44.45" x2="-20.32" y2="39.12" width="0" layer="19" extent="1-1"/>
-<wire x1="-22.86" y1="3.175" x2="-20.32" y2="39.12" width="0" layer="19" extent="1-1"/>
-</signal>
 <signal name="N$3">
 <contactref element="U$1" pad="P$5"/>
 <contactref element="R1" pad="2"/>
-<contactref element="G1" pad="+"/>
-<contactref element="C1" pad="1"/>
-<wire x1="-17.78" y1="52.07" x2="-13.97" y2="58.42" width="0" layer="19" extent="1-1"/>
-<wire x1="-27.69" y1="31.75" x2="-17.78" y2="52.07" width="0" layer="19" extent="1-1"/>
-<wire x1="-17.78" y1="20.955" x2="-27.69" y2="31.75" width="0" layer="19" extent="1-1"/>
+<wire x1="-27.69" y1="31.75" x2="-13.97" y2="58.42" width="0" layer="19" extent="1-1"/>
 </signal>
 <signal name="N$4">
@@
 <wire x1="-39.37" y1="44.45" x2="-19.05" y2="39.12" width="0" layer="19" extent="1-1"/>
 </signal>
+<signal name="N$10">
+<contactref element="JP1" pad="2"/>
+<contactref element="U$1" pad="P$28"/>
+<wire x1="-36.83" y1="44.45" x2="-20.32" y2="39.12" width="0" layer="19" extent="1-1"/>
+</signal>
 </signals>
