File: Circuits/Eagle/Input.sch (EAGLE design)
At the start: 7 parts

Commit message: KiCAD,EAGLEでのPCB設計を試行中。
Parts:
- removed C1: 0.22F, capacitor-wima:C2,5-3
Connections:
- removed net N$1: C1.2, G1.-, JP1.2, U$1.P$28
- new net N$10: JP1.2, U$1.P$28
- net N$3: no longer C1.1, G1.+
Other:
- moved on the sheet: G1, JP1
Changed lines of the file:
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@@
 <part name="S1" library="switch-reed" deviceset="REED-SWITCH-" device="MK6-5-C"/>
 <part name="R1" library="resistor" deviceset="R-US_" device="V234/12" value="1M"/>
-<part name="C1" library="capacitor-wima" deviceset="C" device="2,5-3" value="0.22F"/>
 <part name="SV2" library="con-lstb" deviceset="MA05-1" device="" value="ISP"/>
 <part name="JP1" library="pinhead" deviceset="PINHD-1X2" device="" value="CFG"/>
@@
 <instances>
 <instance part="U$1" gate="G$1" x="48.26" y="40.64"/>
-<instance part="G1" gate="1" x="40.64" y="81.28" rot="R180"/>
+<instance part="G1" gate="1" x="5.08" y="45.72" rot="R90"/>
 <instance part="S1" gate="G$1" x="81.28" y="10.16" rot="R90"/>
 <instance part="R1" gate="G$1" x="17.78" y="35.56" rot="R90"/>
-<instance part="C1" gate="G$1" x="40.64" y="71.12" rot="R90"/>
 <instance part="SV2" gate="G$1" x="104.14" y="55.88" rot="R180"/>
-<instance part="JP1" gate="G$1" x="83.82" y="83.82" rot="R90"/>
+<instance part="JP1" gate="G$1" x="73.66" y="81.28" rot="R270"/>
 </instances>
 <busses>
 </busses>
 <nets>
-<net name="N$1" class="0">
-<segment>
-<pinref part="C1" gate="G$1" pin="2"/>
-<pinref part="U$1" gate="G$1" pin="P$28"/>
-<wire x1="45.72" y1="71.12" x2="50.8" y2="71.12" width="0.1524" layer="91"/>
-<wire x1="50.8" y1="71.12" x2="50.8" y2="66.04" width="0.1524" layer="91"/>
-<pinref part="G1" gate="1" pin="-"/>
-<wire x1="45.72" y1="81.28" x2="50.8" y2="81.28" width="0.1524" layer="91"/>
-<wire x1="50.8" y1="81.28" x2="50.8" y2="71.12" width="0.1524" layer="91"/>
-<junction x="50.8" y="71.12"/>
-<pinref part="JP1" gate="G$1" pin="2"/>
-<wire x1="83.82" y1="81.28" x2="83.82" y2="71.12" width="0.1524" layer="91"/>
-<wire x1="83.82" y1="71.12" x2="50.8" y2="71.12" width="0.1524" layer="91"/>
-<junction x="50.8" y="66.04"/>
-<junction x="83.82" y="81.28"/>
-<junction x="45.72" y="81.28"/>
-<junction x="45.72" y="71.12"/>
-</segment>
-</net>
 <net name="N$3" class="0">
 <segment>
@@
 <pinref part="R1" gate="G$1" pin="2"/>
 <wire x1="25.4" y1="40.64" x2="17.78" y2="40.64" width="0.1524" layer="91"/>
-<wire x1="17.78" y1="40.64" x2="17.78" y2="71.12" width="0.1524" layer="91"/>
-<pinref part="G1" gate="1" pin="+"/>
-<wire x1="17.78" y1="71.12" x2="17.78" y2="81.28" width="0.1524" layer="91"/>
-<wire x1="17.78" y1="81.28" x2="35.56" y2="81.28" width="0.1524" layer="91"/>
-<pinref part="C1" gate="G$1" pin="1"/>
-<wire x1="38.1" y1="71.12" x2="17.78" y2="71.12" width="0.1524" layer="91"/>
-<junction x="17.78" y="71.12"/>
+<wire x1="17.78" y1="40.64" x2="17.78" y2="81.28" width="0.1524" layer="91"/>
 <junction x="17.78" y="40.64"/>
 <junction x="25.4" y="40.64"/>
-<junction x="35.56" y="81.28"/>
-<junction x="38.1" y="71.12"/>
 </segment>
 </net>
@@
 <segment>
 <pinref part="JP1" gate="G$1" pin="1"/>
-<wire x1="81.28" y1="81.28" x2="53.34" y2="81.28" width="0.1524" layer="91"/>
+<wire x1="76.2" y1="83.82" x2="76.2" y2="71.12" width="0.1524" layer="91"/>
+<wire x1="76.2" y1="71.12" x2="53.34" y2="71.12" width="0.1524" layer="91"/>
 <pinref part="U$1" gate="G$1" pin="M3"/>
-<wire x1="53.34" y1="81.28" x2="53.34" y2="66.04" width="0.1524" layer="91"/>
+<wire x1="53.34" y1="71.12" x2="53.34" y2="66.04" width="0.1524" layer="91"/>
 <junction x="53.34" y="66.04"/>
-<junction x="81.28" y="81.28"/>
+<junction x="76.2" y="83.82"/>
 </segment>
 </net>
+<net name="N$10" class="0">
+<segment>
+<pinref part="JP1" gate="G$1" pin="2"/>
+<junction x="73.66" y="83.82"/>
+<wire x1="73.66" y1="83.82" x2="50.8" y2="83.82" width="0.1524" layer="91"/>
+<pinref part="U$1" gate="G$1" pin="P$28"/>
+<wire x1="50.8" y1="83.82" x2="50.8" y2="66.04" width="0.1524" layer="91"/>
+<junction x="50.8" y="66.04"/>
+</segment>
+</net>
