File: Circuits/Input/Input.sch (KiCad schematic (older format))
At the start: 7 parts, among them CN1 WRITER, U1 TWE-Lite_SMD

Commit message: Fixed: Reed switch was not connected to GND.
Connections:
- net labels removed: PULLUP
- wire segments 40 -> 39
- no-connect marks 23 -> 24
Changed lines of the file:
@@
 LIBS:valves
 LIBS:relays
-LIBS:Input-cache
 EELAYER 27 0
 EELAYER END
@@
 Sheet 1 1
 Title "DoorChecker EndPoint_Input"
-Date "20 jan 2015"
+Date "21 jan 2015"
 Rev ""
 Comp "true-nature"
@@
 L SPST REED1
 U 1 1 54360F03
-P 5250 5000
-F 0 "REED1" H 5250 5100 70  0000 C CNN
-F 1 "SPST" H 5250 4900 70  0000 C CNN
-F 2 "~" H 5250 5000 60  0000 C CNN
-F 3 "~" H 5250 5000 60  0000 C CNN
-	1    5250 5000
+P 6450 5950
+F 0 "REED1" H 6450 6050 70  0000 C CNN
+F 1 "SPST" H 6450 5850 70  0000 C CNN
+F 2 "~" H 6450 5950 60  0000 C CNN
+F 3 "~" H 6450 5950 60  0000 C CNN
+	1    6450 5950
 	1    0    0    -1
 $EndComp
@@
 L R R1
 U 1 1 54360F12
-P 4650 4350
-F 0 "R1" V 4730 4350 40  0000 C CNN
-F 1 "2M" V 4657 4351 40  0000 C CNN
-F 2 "~" V 4580 4350 30  0000 C CNN
-F 3 "~" H 4650 4350 30  0000 C CNN
-	1    4650 4350
-	-1   0    0    1
+P 5250 5000
+F 0 "R1" V 5330 5000 40  0000 C CNN
+F 1 "2M" V 5257 5001 40  0000 C CNN
+F 2 "~" V 5180 5000 30  0000 C CNN
+F 3 "~" H 5250 5000 30  0000 C CNN
+	1    5250 5000
+	0    1    1    0
 $EndComp
 $Comp
@@
 L GND #PWR04
 U 1 1 543B5A81
-P 7000 6050
-F 0 "#PWR04" H 7000 6050 30  0001 C CNN
-F 1 "GND" H 7000 5980 30  0001 C CNN
-F 2 "" H 7000 6050 60  0000 C CNN
-F 3 "" H 7000 6050 60  0000 C CNN
-	1    7000 6050
+P 7000 6200
+F 0 "#PWR04" H 7000 6200 30  0001 C CNN
+F 1 "GND" H 7000 6130 30  0001 C CNN
+F 2 "" H 7000 6200 60  0000 C CNN
+F 3 "" H 7000 6200 60  0000 C CNN
+	1    7000 6200
 	1    0    0    -1
 $EndComp
@@
 $EndComp
 Wire Wire Line
-	4650 4600 4650 5000
-Wire Wire Line
-	4650 5000 4750 5000
+	4650 1350 4650 5000
+Wire Wire Line
+	4650 5000 5000 5000
 Wire Wire Line
 	6900 3500 7100 3500
@@
 	6900 3600 7000 3600
 Wire Wire Line
-	7000 2350 7000 6050
+	7000 3600 7000 6200
 Wire Wire Line
 	7000 5800 7700 5800
@@
 Wire Wire Line
 	4650 3600 4800 3600
-Wire Wire Line
-	4650 1350 4650 4100
 Connection ~ 4650 3600
 Wire Wire Line
@@
 	2800 2900 2800 3200
 Wire Wire Line
-	5900 4600 5900 5000
-Wire Wire Line
-	5900 5000 5750 5000
+	5900 4600 5900 5950
+Wire Wire Line
+	5500 5000 5900 5000
 Connection ~ 7000 5800
-Wire Wire Line
-	7000 2350 5900 2350
-Connection ~ 7000 3600
 $Comp
 L PWR_FLAG #FLG05
@@
 	1    0    0    -1
 $EndComp
-Wire Wire Line
-	5900 2350 5900 2500
 Wire Wire Line
 	6000 2500 6000 2200
@@
 Text Label 5800 5000 0    60   ~ 0
 DOOR
-Text Label 4650 5000 0    60   ~ 0
-PULLUP
 Wire Wire Line
 	2800 2100 2800 2300
@@
 	1    0    0    -1
 $EndComp
+Wire Wire Line
+	6950 5950 7000 5950
+Connection ~ 7000 5950
+Wire Wire Line
+	5900 5950 5950 5950
+Connection ~ 5900 5000
+NoConn ~ 5900 2500
 $EndSCHEMATC

Commit message: Set inhibit area under CR2032.
Parts:
- removed CN1: WRITER, ~, symbol CONN_7
- added P1: WRITER-VCC, ~, symbol WRITER-VCC
Connections:
- net labels added: RXD, TXD
- net labels removed: RX, TX
- wire segments 39 -> 40

Commit message: Replaced a EDLC to an array of MLCC.
Parts:
- removed U1: TWE-Lite_SMD, symbol LITE_LITE
- added C2, C3, C4, C5: 100u, ~, symbol CP1
- added U1: TWE_LITE_SMD, MODULE, symbol TWE_LITE_SMD
- C1: value 0.22 -> 100u
Connections:
- net labels added: DI1
- wire segments 40 -> 54
- no-connect marks 24 -> 15

Commit message: Added a voltage monitor.
Parts:
- added Q1: MOS_N, ~, symbol MOS_N
- added R3, R4: 10M, ~, symbol R
- added U2: TCM809RVNB, ~, symbol TCM809RVNB
Connections:
- net labels added: DO1, QGND
- wire segments 54 -> 65
- no-connect marks 15 -> 14

Commit message: Fixed: Switch to configuration mode by M2.
Changed lines of the file:
@@
 Sheet 1 1
 Title "DoorChecker EndPoint_Input"
-Date "2 mar 2015"
+Date "8 mar 2015"
 Rev ""
 Comp "true-nature"
@@
 	8700 4950 8300 4950
 Wire Wire Line
-	8300 4950 8300 1750
+	8300 1750 8300 4950
 Text Label 8450 4950 0    60   ~ 0
 Vcc
@@
 $EndComp
 Wire Wire Line
-	8300 1750 3900 1750
+	3900 1750 8300 1750
 Wire Wire Line
 	7550 2100 7600 2100
@@
 	7700 3150 7700 5250
 Wire Wire Line
-	6050 2300 5600 2300
-Wire Wire Line
-	5600 2300 5600 5550
+	5600 2200 5600 5550
 Wire Wire Line
 	5100 5200 5100 4900
@@
 	5100 3400 6050 3400
 NoConn ~ 6050 2100
-NoConn ~ 6050 2200
 NoConn ~ 6050 2800
 Wire Wire Line
@@
 Text Label 4500 3150 0    60   ~ 0
 QGND
+Wire Wire Line
+	6050 2200 5600 2200
+NoConn ~ 6050 2300
 $EndSCHEMATC

Commit message: Changed register value from 75 to 1k.
Parts:
- Q1: value MOS_N -> RUE002N02
- R2: value 75 -> 1k
- SW1: renamed from REED1; value SPST -> MKA-10110
Changed lines of the file:
@@
 $EndDescr
 $Comp
-L SPST REED1
+L SPST SW1
 U 1 1 54360F03
 P 5100 5700
-F 0 "REED1" H 5100 5800 70  0000 C CNN
-F 1 "SPST" H 5100 5600 70  0000 C CNN
+F 0 "SW1" H 5100 5800 70  0000 C CNN
+F 1 "MKA-10110" H 5100 5600 70  0000 C CNN
 F 2 "~" H 5100 5700 60  0000 C CNN
 F 3 "~" H 5100 5700 60  0000 C CNN
@@
 P 1900 1750
 F 0 "R2" V 1980 1750 40  0000 C CNN
-F 1 "75" V 1907 1751 40  0000 C CNN
+F 1 "1k" V 1907 1751 40  0000 C CNN
 F 2 "~" V 1830 1750 30  0000 C CNN
 F 3 "~" H 1900 1750 30  0000 C CNN
@@
 P 4500 2750
 F 0 "U2" H 4550 2950 60  0000 C CNN
-F 1 "TCM809RVNB" H 4800 2560 60  0000 C CNN
+F 1 "TCM809RVNB" H 4550 3050 60  0000 C CNN
 F 2 "~" H 4500 2750 60  0000 C CNN
 F 3 "~" H 4500 2750 60  0000 C CNN
@@
 P 4400 3450
 F 0 "Q1" H 4410 3620 60  0000 R CNN
-F 1 "MOS_N" H 4410 3300 60  0000 R CNN
+F 1 "RUE002N02" H 4450 3700 60  0000 R CNN
 F 2 "~" H 4400 3450 60  0000 C CNN
 F 3 "~" H 4400 3450 60  0000 C CNN

Commit message: Start to edit current KiCad.
Parts:
- removed R4: 10M, ~, symbol R
Connections:
- wire segments 65 -> 63
Changed lines of the file:
@@
 LIBS:relays
 LIBS:Input-cache
-EELAYER 27 0
+EELAYER 25 0
 EELAYER END
 $Descr A4 11693 8268
@@
 	5800 5150 8700 5150
 Wire Wire Line
-	2200 1400 2200 2050
+	2200 1400 2200 2100
 Wire Wire Line
 	1600 2550 1600 2850
@@
 	2450 1500 2200 1500
 Wire Wire Line
-	2200 2550 2200 2450
+	2200 2550 2200 2400
 Wire Wire Line
 	1600 2550 3400 2550
@@
 	8700 4950 8300 4950
 Wire Wire Line
-	8300 1750 8300 4950
+	8300 4950 8300 1750
 Text Label 8450 4950 0    60   ~ 0
 Vcc
@@
 Connection ~ 2200 1500
 Wire Wire Line
-	2150 1750 3400 1750
+	2050 1750 3400 1750
 Connection ~ 2200 1750
 Wire Wire Line
-	1600 1750 1650 1750
+	1600 1750 1750 1750
 Text Label 1600 1850 1    60   ~ 0
 DC3V
@@
 $EndComp
 Wire Wire Line
-	3400 1750 3400 2050
-Wire Wire Line
-	3400 2550 3400 2450
+	3400 1750 3400 2100
+Wire Wire Line
+	3400 2550 3400 2400
 Connection ~ 2200 2550
 Wire Wire Line
-	2500 2450 2500 2550
+	2500 2400 2500 2550
 Connection ~ 2500 2550
 Wire Wire Line
-	2800 2450 2800 2550
+	2800 2400 2800 2550
 Connection ~ 2800 2550
 Wire Wire Line
-	3100 2450 3100 2550
+	3100 2400 3100 2550
 Connection ~ 3100 2550
 Wire Wire Line
-	3100 2050 3100 1750
+	3100 2100 3100 1750
 Connection ~ 3100 1750
 Wire Wire Line
-	2800 2050 2800 1750
+	2800 2100 2800 1750
 Connection ~ 2800 1750
 Wire Wire Line
-	2500 1750 2500 2050
+	2500 1750 2500 2100
 Connection ~ 2500 1750
 $Comp
@@
 $EndComp
 Wire Wire Line
-	3900 1750 8300 1750
+	8300 1750 3900 1750
 Wire Wire Line
 	7550 2100 7600 2100
@@
 	5600 2200 5600 5550
 Wire Wire Line
-	5100 5200 5100 4900
-Wire Wire Line
-	5100 4400 5100 3400
+	5100 5200 5100 4800
+Wire Wire Line
+	5100 4500 5100 3400
 Wire Wire Line
 	5100 3400 6050 3400
@@
 $EndComp
 $Comp
-L R R4
-U 1 1 54F408A1
-P 5000 2150
-F 0 "R4" V 5080 2150 40  0000 C CNN
-F 1 "10M" V 5007 2151 40  0000 C CNN
-F 2 "~" V 4930 2150 30  0000 C CNN
-F 3 "~" H 5000 2150 30  0000 C CNN
-	1    5000 2150
-	1    0    0    -1
-$EndComp
-$Comp
 L R R3
 U 1 1 54F408D3
@@
 $EndComp
 Wire Wire Line
-	3900 1750 3900 1900
-Wire Wire Line
-	5000 1900 5000 1750
-Connection ~ 5000 1750
+	3900 1750 3900 2000
 Wire Wire Line
 	4150 2700 4150 1750
 Connection ~ 4150 1750
-Wire Wire Line
-	5000 2400 5000 2700
 Connection ~ 5900 2700
-Connection ~ 5000 2700
 Wire Wire Line
 	4500 3250 4500 3050
 Wire Wire Line
-	3900 2400 3900 4000
+	3900 2300 3900 4000
 Wire Wire Line
 	3900 3450 4200 3450

Commit message: Modified reset circuit.
Parts:
- removed Q1: RUE002N02, ~, symbol MOS_N
- added R4: 10M, Resistors_SMD:R_0603_HandSoldering, symbol R
- added U3: 2N7002DW, Housings_SOT-23_SOT-143_TSOT-6:SC-70-6_Handsoldering, symbol 2N7002DW
- BT1: footprint ~ -> favorites:PBCS-75
- C1, C2, C3, C4, C5: footprint ~ -> Capacitors_SMD:C_1210_HandSoldering
- P1: footprint ~ -> favorites:WRITE-7P
- R1, R2, R3: footprint ~ -> Resistors_SMD:R_0603_HandSoldering
- SW1: footprint ~ -> favorites:MKA-10110
- U1: footprint MODULE -> favorites:TWE-001L-NC7
- U2: footprint ~ -> Transistors_SMD:sc70
Connections:
- net labels added: RESET#
- net labels removed: DOOR
- wire segments 63 -> 75
