File: Circuits/Input/Input.sch (KiCad schematic (older format))
At the start: 15 parts, among them P1 WRITER-VCC, SW1 MKA-10110, U1 TWE_LITE_SMD, U2 TCM809RVNB, U3 2N7002DW

Commit message: Simplified power supply block.
Parts:
- removed C2, C3, C4, C5: 100u, Capacitors_SMD:C_1210_HandSoldering, symbol CP1
- removed R2: 1k, Resistors_SMD:R_0603_HandSoldering, symbol R
- removed R3, R4: 10M, Resistors_SMD:R_0603_HandSoldering, symbol R
- removed U2: TCM809RVNB, Transistors_SMD:sc70, symbol TCM809RVNB
- removed U3: 2N7002DW, Housings_SOT-23_SOT-143_TSOT-6:SC-70-6_Handsoldering, symbol 2N7002DW
Connections:
- net labels removed: DC3V, DO1, QGND, RESET#, VCC
- wire segments 75 -> 42
- no-connect marks 14 -> 15
