File: Circuits/Input/Input.sch (KiCad schematic (older format))
At the start: 7 parts, among them P1 WRITER-VCC, Q1 Q_Photo_NPN_CE, SW1 MKA-10110, U1 TWE_LITE_SMD

Commit message: Updated libraries
Parts:
- added C1: 100p, Capacitors_SMD:C_0603_HandSoldering, symbol C_Small
- added R2: 100k, Resistors_SMD:R_0603_HandSoldering, symbol R
- Q1: footprint (none) -> Opto-Devices:PhotoDiode_SFH205
- SW1: symbol SPST -> SW_Reed
- renumbered R2 to R3
Connections:
- wire segments 49 -> 56
Changed lines of the file:
@@
 EESchema Schematic File Version 2
 LIBS:favorites
+LIBS:ac-dc
+LIBS:adc-dac
+LIBS:Altera
+LIBS:analog_devices
+LIBS:analog_switches
+LIBS:atmel
+LIBS:audio
+LIBS:Battery_Management
+LIBS:bbd
+LIBS:Bosch
+LIBS:brooktre
+LIBS:Connector
+LIBS:contrib
+LIBS:cypress
+LIBS:dc-dc
+LIBS:Decawave
+LIBS:device
+LIBS:digital-audio
+LIBS:Diode
+LIBS:Display
+LIBS:driver_gate
+LIBS:dsp
+LIBS:DSP_Microchip_DSPIC33
+LIBS:elec-unifil
+LIBS:ESD_Protection
+LIBS:Espressif
+LIBS:ftdi
+LIBS:gennum
+LIBS:Graphic
+LIBS:hc11
+LIBS:infineon
+LIBS:intel
+LIBS:interface
+LIBS:intersil
+LIBS:ir
+LIBS:Lattice
+LIBS:LED
+LIBS:LEM
+LIBS:linear
+LIBS:Logic_CMOS_4000
+LIBS:Logic_CMOS_IEEE
+LIBS:logic_programmable
+LIBS:Logic_TTL_IEEE
+LIBS:maxim
+LIBS:MCU_NXP_Kinetis
+LIBS:MCU_NXP_LPC
+LIBS:MCU_ST_STM32
+LIBS:Mechanical
+LIBS:memory
+LIBS:microchip
+LIBS:microcontrollers
+LIBS:modules
+LIBS:Motor
+LIBS:motor_drivers
+LIBS:motorola
+LIBS:nordicsemi
+LIBS:nxp
+LIBS:onsemi
+LIBS:opto
+LIBS:Oscillators
+LIBS:philips
 LIBS:power
-LIBS:device
-LIBS:transistors
-LIBS:conn
-LIBS:linear
+LIBS:Power_Management
+LIBS:powerint
+LIBS:pspice
+LIBS:references
 LIBS:regul
-LIBS:74xx
-LIBS:cmos4000
-LIBS:adc-dac
-LIBS:memory
-LIBS:xilinx
-LIBS:microcontrollers
-LIBS:dsp
-LIBS:microchip
-LIBS:analog_switches
-LIBS:motorola
+LIBS:Relay
+LIBS:RF_Bluetooth
+LIBS:rfcom
+LIBS:RFSolutions
+LIBS:Sensor_Current
+LIBS:Sensor_Humidity
+LIBS:sensors
+LIBS:silabs
+LIBS:siliconi
+LIBS:supertex
+LIBS:Switch
 LIBS:texas
-LIBS:intel
-LIBS:audio
-LIBS:interface
-LIBS:digital-audio
-LIBS:philips
-LIBS:display
-LIBS:cypress
-LIBS:siliconi
-LIBS:opto
-LIBS:atmel
-LIBS:contrib
-LIBS:valves
-LIBS:relays
+LIBS:Transformer
+LIBS:Transistor
+LIBS:triac_thyristor
+LIBS:Valve
+LIBS:video
+LIBS:wiznet
+LIBS:Worldsemi
+LIBS:Xicor
+LIBS:zetex
+LIBS:Zilog
 LIBS:Input-cache
 EELAYER 25 0
@@
 $EndDescr
 $Comp
-L SPST SW1
+L SW_Reed SW1
 U 1 1 54360F03
-P 5600 4450
-F 0 "SW1" H 5600 4550 70  0000 C CNN
-F 1 "MKA-10110" H 5600 4350 70  0000 C CNN
-F 2 "favorites:MKA-10110" H 5600 4450 60  0000 C CNN
-F 3 "~" H 5600 4450 60  0000 C CNN
-	1    5600 4450
+P 5600 3950
+F 0 "SW1" H 5600 4050 70  0000 C CNN
+F 1 "MKA-10110" H 5600 3850 70  0000 C CNN
+F 2 "favorites:MKA-10110" H 5600 3950 60  0001 C CNN
+F 3 "~" H 5600 3950 60  0000 C CNN
+	1    5600 3950
 	0    -1   -1   0
 $EndComp
@@
 L R R1
 U 1 1 54360F12
-P 5600 3700
-F 0 "R1" V 5680 3700 40  0000 C CNN
-F 1 "2M" V 5607 3701 40  0000 C CNN
-F 2 "Resistors_SMD:R_0603_HandSoldering" V 5530 3700 30  0000 C CNN
-F 3 "~" H 5600 3700 30  0000 C CNN
-	1    5600 3700
+P 5600 4750
+F 0 "R1" V 5680 4750 40  0000 C CNN
+F 1 "2M" V 5607 4751 40  0000 C CNN
+F 2 "Resistors_SMD:R_0603_HandSoldering" V 5530 4750 30  0001 C CNN
+F 3 "~" H 5600 4750 30  0000 C CNN
+	1    5600 4750
 	1    0    0    -1
 $EndComp
@@
 F 0 "BT1" H 4450 2350 50  0000 C CNN
 F 1 "CR2032" H 4450 1960 50  0000 C CNN
-F 2 "favorites:PBCS-75" H 4450 2150 60  0000 C CNN
+F 2 "favorites:PBCS-75" H 4450 2150 60  0001 C CNN
 F 3 "~" H 4450 2150 60  0000 C CNN
 	1    4450 2150
@@
 F 0 "P1" V 9300 4800 60  0000 C CNN
 F 1 "WRITER-VCC" V 9400 4800 60  0000 C CNN
-F 2 "favorites:WRITE-7P" H 9150 4750 60  0000 C CNN
+F 2 "favorites:WRITE-7P" H 9150 4750 60  0001 C CNN
 F 3 "~" H 9150 4750 60  0000 C CNN
 	1    9200 4800
@@
 NoConn ~ 8050 2500
 $Comp
-L R R2
+L R R3
 U 1 1 587D4FBE
 P 8900 1950
-F 0 "R2" V 8980 1950 40  0000 C CNN
+F 0 "R3" V 8980 1950 40  0000 C CNN
 F 1 "100k" V 8907 1951 40  0000 C CNN
-F 2 "Resistors_SMD:R_0603_HandSoldering" V 8830 1950 30  0000 C CNN
+F 2 "Resistors_SMD:R_0603_HandSoldering" V 8830 1950 30  0001 C CNN
 F 3 "~" H 8900 1950 30  0000 C CNN
 	1    8900 1950
@@
 F 0 "Q1" H 9000 2500 50  0000 L CNN
 F 1 "Q_Photo_NPN_CE" H 9000 2400 50  0000 L CNN
-F 2 "" H 9000 2550 50  0000 C CNN
+F 2 "Opto-Devices:PhotoDiode_SFH205" H 9000 2550 50  0000 C CNN
 F 3 "" H 8800 2450 50  0000 C CNN
 	1    8800 2450
@@
 	6000 1650 6000 3150
 Connection ~ 5900 1750
-Connection ~ 8400 1750
+Connection ~ 8500 1750
 Wire Wire Line
 	8900 1750 8900 1800
@@
 	8900 2100 8900 2250
 Wire Wire Line
-	8900 2700 8900 2650
+	8900 2650 8900 2900
 Wire Wire Line
 	8050 2700 8900 2700
@@
 	6100 5100 8800 5100
 Wire Wire Line
-	8400 4500 8800 4500
-Wire Wire Line
-	8400 1750 8400 4500
+	8500 4500 8800 4500
+Wire Wire Line
+	8500 1750 8500 4500
 Wire Wire Line
 	4450 1750 8900 1750
@@
 Connection ~ 8100 3700
 Wire Wire Line
-	8100 3800 8050 3800
+	8050 3800 8350 3800
 Wire Wire Line
 	8200 3150 8200 4800
@@
 	6100 2200 6100 5100
 Wire Wire Line
-	5600 3950 5600 3850
-Wire Wire Line
-	5600 3550 5600 3400
+	5600 3750 5600 3400
 Wire Wire Line
 	5600 3400 6550 3400
@@
 	6550 2200 6100 2200
 Wire Wire Line
-	5600 5000 5600 4950
+	5600 5000 5600 4900
 Wire Wire Line
 	6400 4600 8800 4600
@@
 	6550 2950 5150 2950
 Connection ~ 5150 2950
+Wire Wire Line
+	5600 4150 5600 4600
+$Comp
+L R R2
+U 1 1 5A82DDEB
+P 8900 3050
+F 0 "R2" V 8980 3050 40  0000 C CNN
+F 1 "100k" V 8907 3051 40  0000 C CNN
+F 2 "Resistors_SMD:R_0603_HandSoldering" V 8830 3050 30  0001 C CNN
+F 3 "~" H 8900 3050 30  0000 C CNN
+	1    8900 3050
+	1    0    0    -1
+$EndComp
+Connection ~ 8900 2700
+Wire Wire Line
+	5600 4500 6800 4500
+Wire Wire Line
+	6800 4500 6800 4000
+Wire Wire Line
+	6800 4000 8900 4000
+Wire Wire Line
+	8900 4000 8900 3200
+Connection ~ 5600 4500
+$Comp
+L C_Small C1
+U 1 1 5A845ABD
+P 8350 3600
+F 0 "C1" H 8360 3670 50  0000 L CNN
+F 1 "100p" H 8360 3520 50  0000 L CNN
+F 2 "Capacitors_SMD:C_0603_HandSoldering" H 8350 3600 50  0001 C CNN
+F 3 "" H 8350 3600 50  0001 C CNN
+	1    8350 3600
+	1    0    0    -1
+$EndComp
+Wire Wire Line
+	8350 3800 8350 3700
+Wire Wire Line
+	8350 3500 8350 3400
+Wire Wire Line
+	8350 3400 8500 3400
+Connection ~ 8500 3400
 $EndSCHEMATC

Commit message: Replaced sensor to pinheader
Parts:
- C1: value 100p -> 1uF; footprint Capacitors_SMD:C_0603_HandSoldering -> Capacitors_SMD:C_0805_HandSoldering
- J1: renamed from Q1; value Q_Photo_NPN_CE -> sensor; footprint Opto-Devices:PhotoDiode_SFH205 -> Connect:PINHEAD1-2; symbol Q_Photo_NPN_CE -> Conn_01x02
Connections:
- wire segments 56 -> 54
Changed lines of the file:
@@
 L R R3
 U 1 1 587D4FBE
-P 8900 1950
-F 0 "R3" V 8980 1950 40  0000 C CNN
-F 1 "100k" V 8907 1951 40  0000 C CNN
-F 2 "Resistors_SMD:R_0603_HandSoldering" V 8830 1950 30  0001 C CNN
-F 3 "~" H 8900 1950 30  0000 C CNN
-	1    8900 1950
+P 8800 1750
+F 0 "R3" V 8880 1750 40  0000 C CNN
+F 1 "100k" V 8807 1751 40  0000 C CNN
+F 2 "Resistors_SMD:R_0603_HandSoldering" V 8730 1750 30  0001 C CNN
+F 3 "~" H 8800 1750 30  0000 C CNN
+	1    8800 1750
+	0    1    1    0
+$EndComp
+$Comp
+L Conn_01x02 J1
+U 1 1 587D57BC
+P 9250 2400
+F 0 "J1" H 9450 2450 50  0000 L CNN
+F 1 "sensor" H 9450 2350 50  0000 L CNN
+F 2 "Connect:PINHEAD1-2" H 9450 2500 50  0000 C CNN
+F 3 "" H 9250 2400 50  0000 C CNN
+	1    9250 2400
 	1    0    0    -1
 $EndComp
 $Comp
-L Q_Photo_NPN_CE Q1
-U 1 1 587D57BC
-P 8800 2450
-F 0 "Q1" H 9000 2500 50  0000 L CNN
-F 1 "Q_Photo_NPN_CE" H 9000 2400 50  0000 L CNN
-F 2 "Opto-Devices:PhotoDiode_SFH205" H 9000 2550 50  0000 C CNN
-F 3 "" H 8800 2450 50  0000 C CNN
-	1    8800 2450
+L R R2
+U 1 1 5A82DDEB
+P 9050 3050
+F 0 "R2" V 9130 3050 40  0000 C CNN
+F 1 "100k" V 9057 3051 40  0000 C CNN
+F 2 "Resistors_SMD:R_0603_HandSoldering" V 8980 3050 30  0001 C CNN
+F 3 "~" H 9050 3050 30  0000 C CNN
+	1    9050 3050
 	1    0    0    -1
 $EndComp
-Connection ~ 8900 2200
+$Comp
+L C_Small C1
+U 1 1 5A845ABD
+P 8350 3600
+F 0 "C1" H 8360 3670 50  0000 L CNN
+F 1 "1uF" H 8360 3520 50  0000 L CNN
+F 2 "Capacitors_SMD:C_0805_HandSoldering" H 8350 3600 50  0001 C CNN
+F 3 "" H 8350 3600 50  0001 C CNN
+	1    8350 3600
+	1    0    0    -1
+$EndComp
 Wire Wire Line
-	8900 2200 9150 2200
-Wire Wire Line
-	9150 2200 9150 1650
-Wire Wire Line
-	9150 1650 6000 1650
+	9050 1650 6000 1650
 Wire Wire Line
 	6000 1650 6000 3150
@@
 Connection ~ 8500 1750
 Wire Wire Line
-	8900 1750 8900 1800
+	9050 2500 9050 2900
 Wire Wire Line
-	8900 2100 8900 2250
-Wire Wire Line
-	8900 2650 8900 2900
-Wire Wire Line
-	8050 2700 8900 2700
+	8050 2700 9050 2700
 Connection ~ 5150 3050
 Wire Wire Line
@@
 	8500 1750 8500 4500
 Wire Wire Line
-	4450 1750 8900 1750
+	4450 1750 8650 1750
 Wire Wire Line
 	8100 2100 8050 2100
@@
 Wire Wire Line
 	5600 4150 5600 4600
-$Comp
-L R R2
-U 1 1 5A82DDEB
-P 8900 3050
-F 0 "R2" V 8980 3050 40  0000 C CNN
-F 1 "100k" V 8907 3051 40  0000 C CNN
-F 2 "Resistors_SMD:R_0603_HandSoldering" V 8830 3050 30  0001 C CNN
-F 3 "~" H 8900 3050 30  0000 C CNN
-	1    8900 3050
-	1    0    0    -1
-$EndComp
-Connection ~ 8900 2700
+Connection ~ 9050 2700
 Wire Wire Line
 	5600 4500 6800 4500
@@
 	6800 4500 6800 4000
 Wire Wire Line
-	6800 4000 8900 4000
+	6800 4000 9050 4000
 Wire Wire Line
-	8900 4000 8900 3200
+	9050 4000 9050 3200
 Connection ~ 5600 4500
-$Comp
-L C_Small C1
-U 1 1 5A845ABD
-P 8350 3600
-F 0 "C1" H 8360 3670 50  0000 L CNN
-F 1 "100p" H 8360 3520 50  0000 L CNN
-F 2 "Capacitors_SMD:C_0603_HandSoldering" H 8350 3600 50  0001 C CNN
-F 3 "" H 8350 3600 50  0001 C CNN
-	1    8350 3600
-	1    0    0    -1
-$EndComp
 Wire Wire Line
 	8350 3800 8350 3700
@@
 	8350 3400 8500 3400
 Connection ~ 8500 3400
+Wire Wire Line
+	8950 1750 9050 1750
+Connection ~ 9050 1750
+Wire Wire Line
+	9050 2400 9050 1650
 $EndSCHEMATC

Commit message: Migrating to KiCad 5.0
Parts:
- removed U1: TWE_LITE_SMD, favorites:TWE-001L-NC7, symbol TWE_LITE_SMD
- added U1: TWELITE_SMD, RF_Module:TWELITE_SMD, symbol RF_ZigBee:TWELITE_SMD
- BT1: symbol BATTERY -> Input-rescue:BATTERY-RESCUE-Input
- C1: footprint Capacitors_SMD:C_0805_HandSoldering -> Capacitor_SMD:C_0603_1608Metric_Pad0.84x1.00mm_HandSolder; symbol C_Small -> device:C_Small
- J1: footprint Connect:PINHEAD1-2 -> Connector_PinHeader_2.54mm:PinHeader_2x01_P2.54mm_Vertical; symbol Conn_01x02 -> Connector:Conn_01x02
- P1: symbol WRITER-VCC -> favorites:WRITER-VCC
- R1, R2, R3: footprint Resistors_SMD:R_0603_HandSoldering -> Resistor_SMD:R_0603_1608Metric_Pad0.84x1.00mm_HandSolder; symbol R -> device:R
- SW1: symbol SW_Reed -> Switch1:SW_Reed
Connections:
- wire segments 54 -> 70

Commit message: Removed rescue library
Parts:
- BT1: symbol Input-rescue:BATTERY-RESCUE-Input -> Device:Battery_Cell
- C1: symbol device:C_Small -> Device:C_Small
- J1: symbol Connector:Conn_01x02 -> Connector_Generic:Conn_01x02
- R1, R2, R3: symbol device:R -> Device:R
- SW1: symbol Switch1:SW_Reed -> Switch:SW_Reed
Changed lines of the file:
@@
 Sheet 1 1
 Title "DoorChecker EndPoint_Input"
-Date "8 mar 2015"
+Date "2018-03-09"
 Rev ""
-Comp "true-nature"
+Comp "https://github.com/true-nature"
 Comment1 ""
 Comment2 ""
@@
 $EndDescr
 $Comp
-L Switch1:SW_Reed SW1
+L Switch:SW_Reed SW1
 U 1 1 54360F03
 P 5600 3950
@@
 $EndComp
 $Comp
-L device:R R1
+L Device:R R1
 U 1 1 54360F12
 P 5600 4750
@@
 $EndComp
 $Comp
-L power1:GND #PWR01
+L power:GND #PWR01
 U 1 1 543B58C8
 P 4450 2700
@@
 $EndComp
 $Comp
-L Input-rescue:BATTERY-RESCUE-Input BT1
+L Device:Battery_Cell BT1
 U 1 1 543B60F0
 P 4450 2150
-F 0 "BT1" H 4450 2350 50  0000 C CNN
-F 1 "CR2032" H 4450 1960 50  0000 C CNN
+F 0 "BT1" H 4350 2300 50  0000 C CNN
+F 1 "CR2032" H 4300 2100 50  0000 C CNN
 F 2 "favorites:PBCS-75" H 4450 2150 60  0001 C CNN
 F 3 "~" H 4450 2150 60  0000 C CNN
 	1    4450 2150
-	0    1    1    0
-$EndComp
-$Comp
-L power1:PWR_FLAG #FLG02
+	1    0    0    -1
+$EndComp
+$Comp
+L power:PWR_FLAG #FLG02
 U 1 1 5486A030
 P 4450 1600
@@
 PRG
 $Comp
-L power1:PWR_FLAG #FLG03
+L power:PWR_FLAG #FLG03
 U 1 1 550F8F4A
 P 4950 4900
@@
 $EndComp
 $Comp
-L device:R R3
+L Device:R R3
 U 1 1 587D4FBE
 P 9500 1750
@@
 $EndComp
 $Comp
-L Connector:Conn_01x02 J1
+L Connector_Generic:Conn_01x02 J1
 U 1 1 587D57BC
 P 9950 2000
@@
 $EndComp
 $Comp
-L device:R R2
+L Device:R R2
 U 1 1 5A82DDEB
 P 9750 3050
@@
 Connection ~ 4450 2550
 Wire Wire Line
-	4450 2450 4450 2550
+	4450 2250 4450 2550
 Wire Wire Line
 	4450 1600 4450 1750
@@
 	5150 3300 5150 5000
 Wire Wire Line
-	4450 1750 4450 1850
+	4450 1750 4450 1950
 Wire Wire Line
 	4450 2550 4450 2700
@@
 	8900 2700 8900 4800
 $Comp
-L device:C_Small C1
+L Device:C_Small C1
 U 1 1 5A845ABD
 P 7900 4350

Commit message: Updated footprint
Other:
- note added: "R1 and R2 are exclusive."
- moved on the sheet: BT1, C1, J1, P1, R1, R2, R3, SW1, U1

Commit message: Updated symbols
Parts:
- U1: symbol RF_ZigBee:TWELITE_SMD -> RF_ZigBee:TWELITE
Changed lines of the file:
@@
-	1    0    0    -1
-$EndComp
-$Comp
-L power:PWR_FLAG #FLG02
-U 1 1 5486A030
-P 1250 1250
-F 0 "#FLG02" H 1250 1345 30  0001 C CNN
-F 1 "PWR_FLAG" H 1250 1430 30  0000 C CNN
-F 2 "" H 1250 1250 60  0000 C CNN
-F 3 "" H 1250 1250 60  0000 C CNN
-	1    1250 1250
 	1    0    0    -1
 $EndComp
@@
 	1    0    0    -1
 $EndComp
-NoConn ~ 3350 1750
+NoConn ~ 3450 1750
 Text Label 2500 2450 0    60   ~ 0
 DI1
-NoConn ~ 3350 1950
+NoConn ~ 3450 1950
 Text Label 6050 4650 0    60   ~ 0
 RST
 Text Label 6050 4850 0    60   ~ 0
 PRG
-$Comp
-L power:PWR_FLAG #FLG03
-U 1 1 550F8F4A
-P 1750 4550
-F 0 "#FLG03" H 1750 4645 50  0001 C CNN
-F 1 "PWR_FLAG" H 1750 4730 50  0000 C CNN
-F 2 "" H 1750 4550 60  0000 C CNN
-F 3 "" H 1750 4550 60  0000 C CNN
-	1    1750 4550
-	1    0    0    -1
-$EndComp
 $Comp
 L Device:R R3
@@
 	6550 1750 6550 1950
 Wire Wire Line
-	5150 1950 6550 1950
+	5050 1950 6550 1950
 Connection ~ 1950 2950
 Wire Wire Line
-	1950 2950 3350 2950
-Connection ~ 1250 1400
+	1950 2950 3450 2950
 Wire Wire Line
 	1250 2200 1950 2200
@@
 	1250 1900 1250 2200
 Wire Wire Line
-	1250 1250 1250 1400
-Wire Wire Line
 	2700 1400 2700 3150
 Wire Wire Line
-	1750 4650 1950 4650
-Wire Wire Line
 	6000 4550 6300 4550
 Wire Wire Line
 	1250 1400 2700 1400
 Wire Wire Line
-	3350 2150 3100 2150
+	3450 2150 3100 2150
 Wire Wire Line
 	3100 2150 3100 4650
 Wire Wire Line
-	5150 2350 5700 2350
+	5050 2350 5700 2350
 Wire Wire Line
 	2900 1850 2900 5150
@@
 	2400 3400 2400 2450
 Wire Wire Line
-	2400 2450 3350 2450
-Wire Wire Line
-	2700 3150 3350 3150
-Wire Wire Line
-	3350 1850 2900 1850
+	2400 2450 3450 2450
+Wire Wire Line
+	2700 3150 3450 3150
+Wire Wire Line
+	3450 1850 2900 1850
 Wire Wire Line
 	2400 4650 2400 4550
@@
 	5700 4850 6300 4850
 Wire Wire Line
-	1750 4550 1750 4650
-Wire Wire Line
 	1950 2200 1950 2850
-Connection ~ 1950 4650
-Wire Wire Line
-	3350 2850 1950 2850
+Wire Wire Line
+	3450 2850 1950 2850
 Connection ~ 1950 2850
 Wire Wire Line
@@
 Wire Wire Line
 	2700 1400 4250 1400
-NoConn ~ 5150 1750
-NoConn ~ 5150 1850
-NoConn ~ 5150 2050
-NoConn ~ 5150 2850
-NoConn ~ 5150 2950
+NoConn ~ 5050 1750
+NoConn ~ 5050 1850
+NoConn ~ 5050 2050
+NoConn ~ 5050 2850
+NoConn ~ 5050 2950
 Wire Wire Line
 	4150 5050 6300 5050
@@
 $EndComp
 Wire Wire Line
-	5150 2750 5300 2750
+	5050 2750 5300 2750
 Wire Wire Line
 	5300 2750 5300 4950
@@
 	5300 4950 6300 4950
 Wire Wire Line
-	5150 2650 5400 2650
+	5050 2650 5400 2650
 Wire Wire Line
 	5400 2650 5400 4750
 Wire Wire Line
 	5400 4750 6300 4750
-NoConn ~ 5150 2150
-NoConn ~ 5150 2250
-NoConn ~ 5150 2450
-NoConn ~ 3350 2250
-Wire Wire Line
-	3350 3050 2800 3050
-NoConn ~ 3350 2550
-NoConn ~ 3350 2650
-NoConn ~ 3350 2750
+NoConn ~ 5050 2150
+NoConn ~ 5050 2250
+NoConn ~ 5050 2450
+NoConn ~ 3450 2250
+Wire Wire Line
+	3450 3050 2800 3050
+NoConn ~ 3450 2550
+NoConn ~ 3450 2650
+NoConn ~ 3450 2750
 Wire Wire Line
 	4250 1450 4250 1400
@@
 	5150 3550 6000 3550
 $Comp
-L RF_ZigBee:TWELITE_SMD U1
+L RF_ZigBee:TWELITE U1
 U 1 1 5A9FFEF1
 P 4250 2450
-F 0 "U1" H 4250 2500 50  0000 C CNN
-F 1 "TWELITE_SMD" H 4300 2350 50  0000 C CNN
+F 0 "U1" H 3800 3300 50  0000 C CNN
+F 1 "TWELITE_SMD" H 4550 3300 50  0000 C CNN
 F 2 "RF_Module:TWELITE_SMD" H 4250 1350 50  0001 C CNN
 F 3 "https://www.mono-wireless.com/jp/products/TWE-LITE/MW-PDS-TWELITE-JP.pdf" H 5000 1450 50  0001 C CNN
@@
 	2400 4000 6550 4000
 Connection ~ 4550 3550
+Connection ~ 1250 1400
+Wire Wire Line
+	1250 1250 1250 1400
+$Comp
+L power:PWR_FLAG #FLG02
+U 1 1 5486A030
+P 1250 1250
+F 0 "#FLG02" H 1250 1345 30  0001 C CNN
+F 1 "PWR_FLAG" H 1250 1430 30  0000 C CNN
+F 2 "" H 1250 1250 60  0000 C CNN
+F 3 "" H 1250 1250 60  0000 C CNN
+	1    1250 1250
+	1    0    0    -1
+$EndComp
+$Comp
+L power:PWR_FLAG #FLG?
+U 1 1 5AAF2C2D
+P 1750 4550
+F 0 "#FLG?" H 1750 4645 30  0001 C CNN
+F 1 "PWR_FLAG" H 1750 4730 30  0000 C CNN
+F 2 "" H 1750 4550 60  0000 C CNN
+F 3 "" H 1750 4550 60  0000 C CNN
+	1    1750 4550
+	1    0    0    -1
+$EndComp
+Wire Wire Line
+	1750 4550 1750 4650
+Wire Wire Line
+	1750 4650 1950 4650
+Connection ~ 1950 4650
 $EndSCHEMATC
