File: Circuits/RainSensor/RainSensor.sch (KiCad schematic (older format))
At the start: 7 parts, among them P1 WRITER-VCC, Q1 Q_Photo_NPN_CE, SW1 MKA-10110, U1 TWE_LITE_SMD

Commit message: 雨センサー基板を作成
Parts:
- removed BT1: CR2032, favorites:PBCS-75, symbol BATTERY
- removed P1: WRITER-VCC, favorites:WRITE-7P, symbol WRITER-VCC
- removed Q1: Q_Photo_NPN_CE, symbol Q_Photo_NPN_CE
- removed R1: 2M, Resistors_SMD:R_0603_HandSoldering, symbol R
- removed R2: 100k, Resistors_SMD:R_0603_HandSoldering, symbol R
- removed SW1: MKA-10110, favorites:MKA-10110, symbol SPST
- removed U1: TWE_LITE_SMD, favorites:TWE-001L-NC7, symbol TWE_LITE_SMD
- added BT?: CR2032, favorites:PBCS-75, symbol BATTERY
- added P?: WRITER-VCC, favorites:WRITE-7P, symbol WRITER-VCC
- added R?: 2M, Resistors_SMD:R_0603_HandSoldering, symbol R
- added R?: 100k, Resistors_SMD:R_0603_HandSoldering, symbol R
- added R?: R_Variable, symbol R_Variable
- added SW?: MKA-10110, favorites:MKA-10110, symbol SPST
- added U?: TWE_LITE_SMD, favorites:TWE-001L-NC7, symbol TWE_LITE_SMD
Connections:
- wire segments 49 -> 64
Changed lines of the file:
@@
 EESchema Schematic File Version 2
-LIBS:favorites
 LIBS:power
 LIBS:device
+LIBS:switches
+LIBS:relays
+LIBS:motors
 LIBS:transistors
 LIBS:conn
@@
 LIBS:contrib
 LIBS:valves
-LIBS:relays
+LIBS:TWE-Lite
+LIBS:favorites
 LIBS:Input-cache
 EELAYER 25 0
@@
 $EndDescr
 $Comp
-L SPST SW1
-U 1 1 54360F03
+L SPST SW?
+U 1 1 5A4B9196
 P 5600 4450
-F 0 "SW1" H 5600 4550 70  0000 C CNN
+F 0 "SW?" H 5600 4550 70  0000 C CNN
 F 1 "MKA-10110" H 5600 4350 70  0000 C CNN
 F 2 "favorites:MKA-10110" H 5600 4450 60  0000 C CNN
@@
 $EndComp
 $Comp
-L R R1
-U 1 1 54360F12
+L R R?
+U 1 1 5A4B9197
 P 5600 3700
-F 0 "R1" V 5680 3700 40  0000 C CNN
+F 0 "R?" V 5680 3700 40  0000 C CNN
 F 1 "2M" V 5607 3701 40  0000 C CNN
 F 2 "Resistors_SMD:R_0603_HandSoldering" V 5530 3700 30  0000 C CNN
@@
 $EndComp
 $Comp
-L GND #PWR01
-U 1 1 543B58C8
+L GND #PWR?
+U 1 1 5A4B9198
 P 4450 2700
-F 0 "#PWR01" H 4450 2700 30  0001 C CNN
+F 0 "#PWR?" H 4450 2700 30  0001 C CNN
 F 1 "GND" H 4450 2630 30  0001 C CNN
 F 2 "" H 4450 2700 60  0000 C CNN
@@
 $EndComp
 $Comp
-L BATTERY BT1
-U 1 1 543B60F0
+L BATTERY BT?
+U 1 1 5A4B9199
 P 4450 2150
-F 0 "BT1" H 4450 2350 50  0000 C CNN
+F 0 "BT?" H 4450 2350 50  0000 C CNN
 F 1 "CR2032" H 4450 1960 50  0000 C CNN
 F 2 "favorites:PBCS-75" H 4450 2150 60  0000 C CNN
@@
 $EndComp
 $Comp
-L PWR_FLAG #FLG02
-U 1 1 5486A030
+L PWR_FLAG #FLG?
+U 1 1 5A4B919A
 P 4450 1600
-F 0 "#FLG02" H 4450 1695 30  0001 C CNN
+F 0 "#FLG?" H 4450 1695 30  0001 C CNN
 F 1 "PWR_FLAG" H 4450 1780 30  0000 C CNN
 F 2 "" H 4450 1600 60  0000 C CNN
@@
 GND
 $Comp
-L WRITER-VCC P1
-U 1 1 54C9BECD
+L WRITER-VCC P?
+U 1 1 5A4B919B
 P 9200 4800
-F 0 "P1" V 9300 4800 60  0000 C CNN
+F 0 "P?" V 9300 4800 60  0000 C CNN
 F 1 "WRITER-VCC" V 9400 4800 60  0000 C CNN
 F 2 "favorites:WRITE-7P" H 9150 4750 60  0000 C CNN
@@
 $EndComp
 $Comp
-L TWE_LITE_SMD U1
-U 1 1 54EABB18
+L TWE_LITE_SMD U?
+U 1 1 5A4B919C
 P 7300 2750
-F 0 "U1" H 7300 2650 50  0000 C CNN
+F 0 "U?" H 7300 2650 50  0000 C CNN
 F 1 "TWE_LITE_SMD" H 7300 3550 50  0000 C CNN
 F 2 "favorites:TWE-001L-NC7" H 7050 1500 50  0001 C CNN
@@
 PRG
 $Comp
-L PWR_FLAG #FLG03
-U 1 1 550F8F4A
+L PWR_FLAG #FLG?
+U 1 1 5A4B919D
 P 4950 4900
-F 0 "#FLG03" H 4950 4995 50  0001 C CNN
+F 0 "#FLG?" H 4950 4995 50  0001 C CNN
 F 1 "PWR_FLAG" H 4950 5080 50  0000 C CNN
 F 2 "" H 4950 4900 60  0000 C CNN
@@
 NoConn ~ 8050 2500
 $Comp
-L R R2
-U 1 1 587D4FBE
+L R R?
+U 1 1 5A4B919E
 P 8900 1950
-F 0 "R2" V 8980 1950 40  0000 C CNN
+F 0 "R?" V 8980 1950 40  0000 C CNN
 F 1 "100k" V 8907 1951 40  0000 C CNN
 F 2 "Resistors_SMD:R_0603_HandSoldering" V 8830 1950 30  0000 C CNN
@@
 	1    0    0    -1
 $EndComp
-$Comp
-L Q_Photo_NPN_CE Q1
-U 1 1 587D57BC
-P 8800 2450
-F 0 "Q1" H 9000 2500 50  0000 L CNN
-F 1 "Q_Photo_NPN_CE" H 9000 2400 50  0000 L CNN
-F 2 "" H 9000 2550 50  0000 C CNN
-F 3 "" H 8800 2450 50  0000 C CNN
-	1    8800 2450
-	1    0    0    -1
-$EndComp
 Connection ~ 8900 2200
 Wire Wire Line
@@
 	8900 1750 8900 1800
 Wire Wire Line
-	8900 2100 8900 2250
-Wire Wire Line
-	8900 2700 8900 2650
+	8900 2100 8900 2200
+Wire Wire Line
+	8900 2200 8900 2250
+Wire Wire Line
+	8900 2700 8900 2550
 Wire Wire Line
 	8050 2700 8900 2700
@@
 Connection ~ 4450 2550
 Wire Wire Line
-	4450 2450 4450 2700
-Wire Wire Line
-	4450 1600 4450 1850
+	4450 2450 4450 2550
+Wire Wire Line
+	4450 2550 4450 2700
+Wire Wire Line
+	4450 1600 4450 1750
+Wire Wire Line
+	4450 1750 4450 1850
 Wire Wire Line
 	5900 1750 5900 3250
 Wire Wire Line
-	4950 5000 8800 5000
+	4950 5000 5150 5000
+Wire Wire Line
+	5150 5000 5600 5000
+Wire Wire Line
+	5600 5000 8100 5000
+Wire Wire Line
+	8100 5000 8800 5000
 Wire Wire Line
 	6200 4900 8800 4900
@@
 	8400 1750 8400 4500
 Wire Wire Line
-	4450 1750 8900 1750
+	4450 1750 5900 1750
+Wire Wire Line
+	5900 1750 8100 1750
+Wire Wire Line
+	8100 1750 8400 1750
+Wire Wire Line
+	8400 1750 8900 1750
 Wire Wire Line
 	8100 2100 8050 2100
@@
 	8100 3400 8050 3400
 Wire Wire Line
-	8100 3400 8100 5000
+	8100 3400 8100 3500
+Wire Wire Line
+	8100 3500 8100 3600
+Wire Wire Line
+	8100 3600 8100 3700
+Wire Wire Line
+	8100 3700 8100 3800
+Wire Wire Line
+	8100 3800 8100 5000
 Wire Wire Line
 	8100 3500 8050 3500
@@
 	4950 4900 4950 5000
 Wire Wire Line
-	5150 2550 5150 5000
+	5150 2550 5150 2950
+Wire Wire Line
+	5150 2950 5150 3050
+Wire Wire Line
+	5150 3050 5150 5000
 Connection ~ 5150 5000
 Wire Wire Line
@@
 	6550 2950 5150 2950
 Connection ~ 5150 2950
+$Comp
+L R_Variable R?
+U 1 1 5A4B9363
+P 8900 2400
+F 0 "R?" V 9000 2300 50  0000 L CNN
+F 1 "R_Variable" V 8800 2350 50  0000 L CNN
+F 2 "" V 8830 2400 50  0001 C CNN
+F 3 "" H 8900 2400 50  0001 C CNN
+	1    8900 2400
+	1    0    0    -1
+$EndComp
 $EndSCHEMATC

Commit message: Replaced SMD by DIP
Parts:
- U?: value TWE_LITE_SMD -> TWE_LITE_DIP; footprint favorites:TWE-001L-NC7 -> Housings_DIP:DIP-28_W15.24mm_Socket; symbol TWE_LITE_SMD -> TWE_LITE_DIP
Changed lines of the file:
@@
 LIBS:TWE-Lite
 LIBS:favorites
-LIBS:Input-cache
+LIBS:RainSensor-cache
 EELAYER 25 0
 EELAYER END
@@
 $EndComp
 $Comp
-L TWE_LITE_SMD U?
+L TWE_LITE_DIP U?
 U 1 1 5A4B919C
 P 7300 2750
 F 0 "U?" H 7300 2650 50  0000 C CNN
-F 1 "TWE_LITE_SMD" H 7300 3550 50  0000 C CNN
-F 2 "favorites:TWE-001L-NC7" H 7050 1500 50  0001 C CNN
+F 1 "TWE_LITE_DIP" H 7300 3550 50  0000 C CNN
+F 2 "Housings_DIP:DIP-28_W15.24mm_Socket" H 7050 1500 50  0001 C CNN
 F 3 "DOCUMENTATION" H 7650 1500 50  0001 C CNN
 	1    7300 2750
